Commit message: work on 10/19
-ben

File: dev_ws/src/description/robot_core.xacro (robot description, xacro)
@@ -1,9 +1,13 @@
 <?xml version="1.0"?>
 <robot xmlns:xacro="http://www.ros.org/wiki/xacro">
-    <material name="grey">
-        <color rgba="1 1 1 0.75" />
+    <xacro:include filename="inertial_marcos.xacro">
+    <material name="white">
+        <color rgba="1 1 1 1" />
+    </material>
+    <material name="blue">
+        <color rgba="0.2 0.2 1 1" />
     </material>
     <material name="black">
-        <color rgba="1 1 1 1" />
+        <color rgba="0 0 0 1" />
     </material>
     <!-- Base Link -->
@@ -14,14 +18,23 @@
         <parent link="base_link"/>
         <child link="chassis"/>
-        <origin xyz="-0.1 0 0"/>
+        <origin xyz="-0.075 0 0"/>
     </joint>
     <link name="chassis">
         <visual>
-        <origin xyz="0.085 0 0.05"/>
+        <origin xyz="0.085 0 0.01"/>
             <geometry>
                 <cylinder radius="0.085" length="0.055"/>
             </geometry>
-            <material name="grey"/>
+            <material name="blue"/>
         </visual>
+        <collision>
+        <origin xyz="0.085 0 0.01"/>
+            <geometry>
+                <cylinder radius="0.085" length="0.055"/>
+            </geometry>
+        </collision>
+        <xacro:inertial_cylinder mass="0.5" radius="0.085" length="0.01">
+            <origin xyz="0.085 0 0.1" rpy="0 0 0"/>
+        </xacro:inertial_cylinder>
     </link>
     <!-- Left Wheel Link -->
@@ -29,5 +42,5 @@
         <parent link="base_link"/>
         <child link="left_wheel"/>
-        <origin xyz="0 0.085 0" rpy="-${pi/2} 0 0"/>
+        <origin xyz="0 0.06 0" rpy="-${pi/2} 0 0"/>
         <axis xyz="0 0 1"/>
     </joint>
@@ -35,8 +48,16 @@
         <visual>
             <geometry>
-                <cylinder radius="0.06" length="0.025"/>
+                <cylinder radius="0.0325" length="0.025"/>
             </geometry>
         <material name="black"/>
         </visual>
+        <collision>
+            <geometry>
+                <cylinder radius="0.0325" length="0.025"/>
+            </geometry>
+        </collision>
+        <xacro:inertial_cylinder mass="0.1" radius="0.0325" length="0.025">
+            <origin xyz="0 0 0" rpy="0 0 0"/>
+        </xacro:inertial_cylinder>
     </link>
         <!-- Right Wheel Link -->
@@ -44,5 +65,5 @@
         <parent link="base_link"/>
         <child link="right_wheel"/>
-        <origin xyz="0 -0.085 0" rpy="${pi/2} 0 0"/>
+        <origin xyz="0 -0.06 0" rpy="${pi/2} 0 0"/>
         <axis xyz="0 0 -1"/>
     </joint>
@@ -50,8 +71,38 @@
         <visual>
             <geometry>
-                <cylinder radius="0.06" length="0.025"/>
+                <cylinder radius="0.0325" length="0.025"/>
             </geometry>
         <material name="black"/>
         </visual>
+        <collision>
+            <geometry>
+                <cylinder radius="0.0325" length="0.025"/>
+            </geometry>
+        </collision>
+        <xacro:inertial_cylinder mass="0.1" radius="0.0325" length="0.025">
+            <origin xyz="0 0 0" rpy="0 0 0"/>
+        </xacro:inertial_cylinder>
+    </link>
+    <!-- Caster Wheel Link -->
+    <joint name="caster_wheel_joint" type="fixed">
+        <parent link="base_link"/>
+        <child link="caster_wheel"/>
+        <origin xyz="0.06 0 -0.0125"/>
+    </joint>
+    <link name="caster_wheel">
+        <visual>
+            <geometry>
+                <sphere radius="0.0225"/>
+            </geometry>
+            <material name="white"/>
+        </visual>
+        <collision>
+            <geometry>
+                <sphere radius="0.0225"/>
+            </geometry>
+        </collision>
+        <xacro:inertial_sphere mass="0.1" radius="0.0225">
+            <origin xyz="0 0 0" rpy="0 0 0"/>
+        </xacro:inertial_sphere>
     </link>
 </robot>

Commit message: can now use gazebo with the launch_sim.launch.py file
-Ben

File: dev_ws/src/description/robot_core.xacro (robot description, xacro)
@@ -38,4 +38,7 @@
         </xacro:inertial_cylinder>
     </link>
+    <gazebo reference="chassis">
+        <material>Gazebo/Blue</material>
+    </gazebo>
     <!-- Left Wheel Link -->
     <joint name="left_wheel_joint" type="continuous">
@@ -61,4 +64,7 @@
         </xacro:inertial_cylinder>
     </link>
+    <gazebo reference="left_wheel">
+        <material>Gazebo/Black</material>
+    </gazebo>
         <!-- Right Wheel Link -->
     <joint name="right_wheel_joint" type="continuous">
@@ -84,4 +90,7 @@
         </xacro:inertial_cylinder>
     </link>
+    <gazebo reference="right_wheel">
+        <material>Gazebo/Black</material>
+    </gazebo>
     <!-- Caster Wheel Link -->
     <joint name="caster_wheel_joint" type="fixed">
@@ -106,3 +115,8 @@
         </xacro:inertial_sphere>
     </link>
+    <gazebo reference="caster_wheel">
+        <material>Gazebo/White</material>
+        <mu1 value="0.001"/>
+        <mu2 value="0.001"/>
+    </gazebo>
 </robot>
